Commit message: refactor: model_color macro  optimisation

File: docker/jetauto/jetauto_simulations/jetauto_description/urdf/depth_camera.gazebo.xacro (robot description, xacro)
@@ -45,10 +45,5 @@
         </sensor>
     </gazebo>
-    <xacro:macro name="model_color" params="link_name color_name">
-        <gazebo reference="${link_name}">
-            <material>Gazebo/${color_name}</material>
-            <turnGravityOff>false</turnGravityOff>
-        </gazebo>
-    </xacro:macro>
-    <xacro:model_color link_name="$(arg depth_camera_name)_link"    color_name="black"/>
+    <xacro:include filename="$(find jetauto_description)/urdf/model_color.xacro"/>
+    <xacro:model_color link_name="$(arg depth_camera_name)_link"    color_name="Black"/>
 </robot>

File: docker/jetauto/jetauto_simulations/jetauto_description/urdf/jetauto_car.gazebo.xacro (robot description, xacro)
@@ -10,18 +10,13 @@
         </plugin>
     </gazebo>
-    <xacro:macro name="model_color" params="link_name color_name">
-        <gazebo reference="${link_name}">
-            <material>Gazebo/${color_name}</material>
-            <turnGravityOff>false</turnGravityOff>
-        </gazebo>
-    </xacro:macro>
-    <xacro:model_color link_name="base_link"                        color_name="green"/>
-    <xacro:model_color link_name="lidar_link"                       color_name="black"/>
-    <xacro:model_color link_name="back_shell_link"                  color_name="black"/>
-    <xacro:model_color link_name="wheel_right_front_link"           color_name="black"/>
-    <xacro:model_color link_name="wheel_left_front_link"            color_name="black"/>
-    <xacro:model_color link_name="wheel_right_back_link"            color_name="black"/>
-    <xacro:model_color link_name="wheel_left_back_link"             color_name="black"/>
-    <xacro:model_color link_name="mic_link"                         color_name="black"/>
-    <xacro:model_color link_name="speaker_link"                     color_name="black"/>
+    <xacro:include filename="$(find jetauto_description)/urdf/model_color.xacro"/>
+    <xacro:model_color link_name="base_link"                        color_name="Green"/>
+    <xacro:model_color link_name="lidar_link"                       color_name="Black"/>
+    <xacro:model_color link_name="back_shell_link"                  color_name="Black"/>
+    <xacro:model_color link_name="wheel_right_front_link"           color_name="Black"/>
+    <xacro:model_color link_name="wheel_left_front_link"            color_name="Black"/>
+    <xacro:model_color link_name="wheel_right_back_link"            color_name="Black"/>
+    <xacro:model_color link_name="wheel_left_back_link"             color_name="Black"/>
+    <xacro:model_color link_name="mic_link"                         color_name="Black"/>
+    <xacro:model_color link_name="speaker_link"                     color_name="Black"/>
 </robot>

File: docker/jetauto/jetauto_simulations/jetauto_description/urdf/materials.xacro (robot description, xacro)
@@ -1,4 +1,4 @@
 <?xml version="1.0"?>
-<robot>
+<robot xmlns:xacro="http://ros.org/wiki/xacro">
     <material name="black">
         <color rgba="0.1 0.1 0.1 1.0"/>

File: docker/jetauto/jetauto_simulations/jetauto_description/urdf/screen.gazebo.xacro (robot description, xacro)
@@ -1,10 +1,5 @@
 <?xml version="1.0" encoding="utf-8" ?>
 <robot xmlns:xacro="http://ros.org/wiki/xacro">
-    <xacro:macro name="model_color" params="link_name color_name">
-        <gazebo reference="${link_name}">
-            <material>Gazebo/${color_name}</material>
-            <turnGravityOff>false</turnGravityOff>
-        </gazebo>
-    </xacro:macro>
-    <xacro:model_color link_name="screen_link"  color_name="black"/>
+    <xacro:include filename="$(find jetauto_description)/urdf/model_color.xacro"/>
+    <xacro:model_color link_name="screen_link"  color_name="Black"/>
 </robot>
